File: kicad/board/board.sch (KiCad schematic (older format))
At the start: 34 parts

Commit message: Update
Parts:
- removed C?: 10uF, symbol Device:CP
- AT_C100U: renamed from C?; value 100nF -> 100uF
- AT_C20P1, AT_C20P2: renamed from C?; value C -> 20pF
- AT_R1: renamed from R?; value R -> 10k
- AT_SW_R: renamed from SW?; value SW_DPST_x2 -> 1
- MV_C1: renamed from C?; value MV_C1 -> 470uF
- SW_CL_Q, SW_OP_Q: renamed from Q?; value Q_NPN_BCE -> BC337
- gave numbers to parts that had none: 5
Connections:
- net PC?: no longer J?.1 (Pin_1), J?.1 (Pin_1), J?.1 (Pin_1), J?.1 (Pin_1), J?.2 (Pin_2), J?.2 (Pin_2), J?.2 (Pin_2), SW_CL_Q.2, SW_OP_R.2, U?.2 (DATA)
- net AT_D11: now reaches U?.11 (PD5)
- net AT_D11: now also SW_OP_R.2
- net AT_D12: now reaches U?.12 (PD6)
- net AT_D12: now also J?.2 (Pin_2), SW_CL_Q.2
- net AT_D13: now reaches U?.13 (PD7)
- net AT_D13: now also J?.2 (Pin_2)
- net AT_D14: now reaches U?.14 (PB0)
- net AT_D14: now also U?.2 (DATA)
- net AT_P2 renamed AT_RX
- net AT_RX: now also J?.1 (Pin_1)
- net AT_P3 renamed AT_TX
- net AT_TX: now also J?.2 (Pin_2)
- net AT_P4 renamed AT_D4
- net AT_D4: now also J?.1 (Pin_1)
- net AT_P5 renamed AT_D5
- net AT_D5: now also J?.1 (Pin_1)
- net AT_P6 renamed AT_D6
- net AT_D6: now also J?.1 (Pin_1)
Changed lines of the file:
@@
 	3100 1950 3550 1950
 $Comp
-L Device:CP C?
+L Device:CP MV_C1
 U 1 1 6241F25B
 P 3250 1400
-F 0 "C?" H 3368 1446 50  0000 L CNN
-F 1 "MV_C1" H 3368 1355 50  0000 L CNN
+F 0 "MV_C1" H 3368 1446 50  0000 L CNN
+F 1 "470uF" H 3368 1355 50  0000 L CNN
 F 2 "" H 3288 1250 50  0001 C CNN
 F 3 "~" H 3250 1400 50  0001 C CNN
@@
 Text GLabel 3550 2400 2    50   Input ~ 0
 GND
-$Comp
-L Device:R R?
-U 1 1 6243205C
-P 7250 3350
-F 0 "R?" V 7043 3350 50  0000 C CNN
-F 1 "R" V 7134 3350 50  0000 C CNN
-F 2 "" V 7180 3350 50  0001 C CNN
-F 3 "~" H 7250 3350 50  0001 C CNN
-	1    7250 3350
-	0    1    1    0
-$EndComp
 Wire Wire Line
 	7400 3350 7650 3350
@@
 V5
 $Comp
-L Switch:SW_DPST_x2 SW?
+L Switch:SW_DPST_x2 AT_SW_R
 U 1 1 62437558
 P 7400 2950
-F 0 "SW?" H 7400 3185 50  0000 C CNN
-F 1 "SW_DPST_x2" H 7400 3094 50  0000 C CNN
+F 0 "AT_SW_R" H 7400 3185 50  0000 C CNN
+F 1 "1" H 7400 3094 50  0001 C CNN
 F 2 "" H 7400 2950 50  0001 C CNN
 F 3 "~" H 7400 2950 50  0001 C CNN
@@
 GND
 Text GLabel 9000 1300 0    50   Input ~ 0
-PC?
+AT_D4
 Wire Wire Line
 	9000 1300 9300 1300
 Text GLabel 6650 3550 2    50   Input ~ 0
-AT_P2
+AT_RX
 Text GLabel 6650 3650 2    50   Input ~ 0
-AT_P3
+AT_TX
 Text GLabel 6650 3750 2    50   Input ~ 0
-AT_P4
+AT_D4
 Text GLabel 6650 3850 2    50   Input ~ 0
-AT_P5
+AT_D5
 Wire Wire Line
 	6500 3550 6650 3550
@@
 	6500 3950 6650 3950
 Text GLabel 6650 3950 2    50   Input ~ 0
-AT_P6
-Wire Wire Line
-	6000 1550 6000 1000
-Wire Wire Line
-	6000 1000 5900 1000
+AT_D6
 Wire Wire Line
 	5900 1550 5900 1000
-Connection ~ 5900 1000
-$Comp
-L Device:CP C?
+$Comp
+L Device:CP AT_C100U
 U 1 1 6245CF8B
 P 5350 1200
-F 0 "C?" H 5150 1150 50  0000 L CNN
-F 1 "100nF" H 5150 1050 50  0000 L CNN
+F 0 "AT_C100U" H 4850 1150 50  0000 L CNN
+F 1 "100uF" H 4950 1050 50  0000 L CNN
 F 2 "" H 5388 1050 50  0001 C CNN
 F 3 "~" H 5350 1200 50  0001 C CNN
@@
 	1    0    0    -1
 $EndComp
-$Comp
-L Device:CP C?
-U 1 1 6245DC54
-P 5650 1200
-F 0 "C?" H 5750 1100 50  0000 L CNN
-F 1 "10uF" H 5700 1000 50  0000 L CNN
-F 2 "" H 5688 1050 50  0001 C CNN
-F 3 "~" H 5650 1200 50  0001 C CNN
-	1    5650 1200
-	1    0    0    -1
-$EndComp
 Wire Wire Line
 	5150 1000 5350 1000
@@
 Connection ~ 5350 1000
 Wire Wire Line
-	5350 1000 5650 1000
-Wire Wire Line
-	5650 1050 5650 1000
-Connection ~ 5650 1000
-Wire Wire Line
-	5650 1000 5900 1000
-Wire Wire Line
-	5650 1350 5650 1500
-Wire Wire Line
-	5650 1500 5350 1500
-Wire Wire Line
 	5350 1350 5350 1500
-Connection ~ 5350 1500
 Wire Wire Line
 	5350 1500 5150 1500
@@
 GND
 $Comp
-L Device:Crystal Y?
+L Device:Crystal AT_XTAL
 U 1 1 62469428
 P 7400 2250
-F 0 "Y?" V 7354 2381 50  0000 L CNN
-F 1 "Crystal" V 7445 2381 50  0000 L CNN
+F 0 "AT_XTAL" V 7354 2381 50  0000 L CNN
+F 1 "Crystal" V 7445 2381 50  0001 L CNN
 F 2 "" H 7400 2250 50  0001 C CNN
 F 3 "~" H 7400 2250 50  0001 C CNN
@@
 	7400 2550 7400 2400
 $Comp
-L Device:C C?
+L Device:C AT_C20P1
 U 1 1 6246C3F2
 P 7750 2550
-F 0 "C?" V 7498 2550 50  0000 C CNN
-F 1 "C" V 7589 2550 50  0000 C CNN
+F 0 "AT_C20P1" V 7498 2550 50  0000 C CNN
+F 1 "20pF" V 7589 2550 50  0000 C CNN
 F 2 "" H 7788 2400 50  0001 C CNN
 F 3 "~" H 7750 2550 50  0001 C CNN
@@
 $EndComp
 $Comp
-L Device:C C?
+L Device:C AT_C20P2
 U 1 1 6246CD91
 P 7750 2050
-F 0 "C?" V 7498 2050 50  0000 C CNN
-F 1 "C" V 7589 2050 50  0000 C CNN
+F 0 "AT_C20P2" V 7498 2050 50  0000 C CNN
+F 1 "20pF" V 7589 2050 50  0000 C CNN
 F 2 "" H 7788 1900 50  0001 C CNN
 F 3 "~" H 7750 2050 50  0001 C CNN
@@
 GND
 Text GLabel 9000 1750 0    50   Input ~ 0
-PC?
+AT_D5
 Wire Wire Line
 	9000 1750 9300 1750
@@
 GND
 Text GLabel 9000 2200 0    50   Input ~ 0
-PC?
+AT_D6
 Wire Wire Line
 	9000 2200 9300 2200
@@
 	9300 900  9000 900
 Text GLabel 9000 800  0    50   Input ~ 0
-PC?
+AT_RX
 Text GLabel 9000 900  0    50   Input ~ 0
-PC?
-$Comp
-L Device:Q_NPN_BCE Q?
+AT_TX
+$Comp
+L Device:Q_NPN_BCE SW_OP_Q
 U 1 1 624AAF7A
 P 8900 4200
-F 0 "Q?" H 9091 4246 50  0000 L CNN
-F 1 "Q_NPN_BCE" H 9091 4155 50  0000 L CNN
+F 0 "SW_OP_Q" H 9091 4246 50  0000 L CNN
+F 1 "BC337" H 9091 4155 50  0000 L CNN
 F 2 "" H 9100 4300 50  0001 C CNN
 F 3 "~" H 8900 4200 50  0001 C CNN
@@
 $EndComp
 $Comp
-L Device:R R?
+L Device:R SW_OP_R
 U 1 1 624AF8C3
 P 8550 4200
-F 0 "R?" V 8343 4200 50  0000 C CNN
+F 0 "SW_OP_R" V 8343 4200 50  0000 C CNN
 F 1 "R" V 8434 4200 50  0000 C CNN
 F 2 "" V 8480 4200 50  0001 C CNN
@@
 $EndComp
 Text GLabel 8400 4200 0    50   Input ~ 0
-PC?
-$Comp
-L Connector:Screw_Terminal_01x02 J?
+AT_D11
+$Comp
+L Connector:Screw_Terminal_01x02 SW_OP_SCREW
 U 1 1 624B041A
 P 9500 3600
-F 0 "J?" H 9580 3592 50  0000 L CNN
-F 1 "Screw_Terminal_01x02" H 9580 3501 50  0000 L CNN
+F 0 "SW_OP_SCREW" H 9580 3592 50  0000 L CNN
+F 1 "Screw_Terminal_01x02" H 9580 3501 50  0001 L CNN
 F 2 "" H 9500 3600 50  0001 C CNN
 F 3 "~" H 9500 3600 50  0001 C CNN
@@
 V12
 $Comp
-L Device:Q_NPN_BCE Q?
+L Device:Q_NPN_BCE SW_CL_Q
 U 1 1 624C4F6D
 P 8900 5600
-F 0 "Q?" H 9091 5646 50  0000 L CNN
-F 1 "Q_NPN_BCE" H 9091 5555 50  0000 L CNN
+F 0 "SW_CL_Q" H 9091 5646 50  0000 L CNN
+F 1 "BC337" H 9091 5555 50  0000 L CNN
 F 2 "" H 9100 5700 50  0001 C CNN
 F 3 "~" H 8900 5600 50  0001 C CNN
@@
 	1    0    0    -1
 $EndComp
-$Comp
-L Device:R R?
-U 1 1 624C4F73
-P 8550 5600
-F 0 "R?" V 8343 5600 50  0000 C CNN
-F 1 "R" V 8434 5600 50  0000 C CNN
-F 2 "" V 8480 5600 50  0001 C CNN
-F 3 "~" H 8550 5600 50  0001 C CNN
-	1    8550 5600
-	0    1    1    0
-$EndComp
 Text GLabel 8400 5600 0    50   Input ~ 0
-PC?
-$Comp
-L Connector:Screw_Terminal_01x02 J?
+AT_D12
+$Comp
+L Connector:Screw_Terminal_01x02 SW_CL_SCREW
 U 1 1 624C4F7A
 P 9500 5000
-F 0 "J?" H 9580 4992 50  0000 L CNN
-F 1 "Screw_Terminal_01x02" H 9580 4901 50  0000 L CNN
+F 0 "SW_CL_SCREW" H 9580 4992 50  0000 L CNN
+F 1 "Screw_Terminal_01x02" H 9580 4901 50  0001 L CNN
 F 2 "" H 9500 5000 50  0001 C CNN
 F 3 "~" H 9500 5000 50  0001 C CNN
@@
 	11850 900  11400 900
 Text GLabel 11400 900  0    50   Input ~ 0
-PC?
+AT_D12
 $Comp
 L Connector:Screw_Terminal_01x02 J?
@@
 	11850 1450 11400 1450
 Text GLabel 11400 1450 0    50   Input ~ 0
-PC?
+AT_D13
 $Comp
 L Own:RF_RX_433MHz U?
@@
 GND
 Text GLabel 11550 2150 0    50   Input ~ 0
-PC?
+AT_D14
 Text GLabel 12250 2050 2    50   Input ~ 0
 V5
@@
 	3550 2400 2800 2400
 Connection ~ 2800 2400
+$Comp
+L Device:R AT_R1
+U 1 1 6243205C
+P 7250 3350
+F 0 "AT_R1" V 7043 3350 50  0000 C CNN
+F 1 "10k" V 7134 3350 50  0001 C CNN
+F 2 "" V 7180 3350 50  0001 C CNN
+F 3 "~" H 7250 3350 50  0001 C CNN
+	1    7250 3350
+	0    1    1    0
+$EndComp
+Wire Wire Line
+	5350 1000 5900 1000
+Wire Wire Line
+	6000 1550 6000 800
+Wire Wire Line
+	6000 800  5150 800
+Text GLabel 5150 800  0    50   Input ~ 0
+V5
+$Comp
+L Device:R SW_CL_Q
+U 1 1 624C4F73
+P 8550 5600
+F 0 "SW_CL_Q" V 8343 5600 50  0000 C CNN
+F 1 "R" V 8434 5600 50  0000 C CNN
+F 2 "" V 8480 5600 50  0001 C CNN
+F 3 "~" H 8550 5600 50  0001 C CNN
+	1    8550 5600
+	0    1    1    0
+$EndComp
+Text GLabel 6650 4050 2    50   Input ~ 0
+AT_D11
+Text GLabel 6650 4150 2    50   Input ~ 0
+AT_D12
+Wire Wire Line
+	6500 4050 6650 4050
+Wire Wire Line
+	6500 4150 6650 4150
+Text GLabel 6650 4250 2    50   Input ~ 0
+AT_D13
+Wire Wire Line
+	6500 4250 6650 4250
+Text GLabel 6650 1850 2    50   Input ~ 0
+AT_D14
+Wire Wire Line
+	6650 1850 6500 1850
 $EndSCHEMATC

Commit message: Update
Parts:
- removed R? (x5): R, symbol Device:R
- added D?: LED, symbol Device:LED
- added R?: 1k, symbol Device:R
Connections:
- net GND: now also J?.1 (Pin_1), J?.2 (Pin_2), J?.2 (Pin_2), J?.2 (Pin_2), J?.2 (Pin_2), J?.2 (Pin_2), R?.1
- net V5: no longer J?.1 (Pin_1)
- net AT_P9: now reaches U?.15 (PB1)
- net AT_P9: now also J?.2 (Pin_2)
- net AT_P10: now reaches U?.16 (PB2)
- net AT_P10: now also J?.2 (Pin_2)
- net AT_P11: now reaches U?.17 (PB3)
- net AT_P11: now also U?.2 (DATA)
- net at U?.19 (PB5): now also D?.2 (A)
- net AT_D11 renamed AT_P5
- net AT_P5: now also J?.1 (Pin_1); no longer SW_OP_R.2
- removed net AT_D12: J?.2 (Pin_2), SW_CL_Q.2, U?.12 (PD6)
- net AT_D13 renamed AT_P7
- net AT_P7: now also SW_OP_R.2; no longer J?.2 (Pin_2)
- net AT_D14 renamed AT_P8
- net AT_P8: now also SW_CL_Q.2; no longer U?.2 (DATA)
- net AT_D4 renamed AT_P2
- net AT_D5 renamed AT_P12
- net AT_D6 renamed AT_P4
- net PC? renamed AT_P6
- net AT_P6: now also U?.12 (PD6); no longer J?.1 (Pin_1)
- new net: D?.1 (K), R?.2
Changed lines of the file:
@@
 	1    0    0    -1
-$EndComp
-$Comp
-L Device:R R?
-U 1 1 62446986
-P 9150 1400
-F 0 "R?" V 8943 1400 50  0000 C CNN
-F 1 "R" V 9034 1400 50  0000 C CNN
-F 2 "" V 9080 1400 50  0001 C CNN
-F 3 "~" H 9150 1400 50  0001 C CNN
-	1    9150 1400
-	0    1    1    0
 $EndComp
 Text GLabel 9000 1400 0    50   Input ~ 0
 GND
 Text GLabel 9000 1300 0    50   Input ~ 0
-AT_D4
+AT_P2
 Wire Wire Line
 	9000 1300 9300 1300
@@
 AT_TX
 Text GLabel 6650 3750 2    50   Input ~ 0
-AT_D4
+AT_P2
 Text GLabel 6650 3850 2    50   Input ~ 0
-AT_D5
+AT_P12
 Wire Wire Line
 	6500 3550 6650 3550
@@
 	6500 3950 6650 3950
 Text GLabel 6650 3950 2    50   Input ~ 0
-AT_D6
+AT_P4
 Wire Wire Line
 	5900 1550 5900 1000
@@
 	1    0    0    -1
 $EndComp
-$Comp
-L Device:R R?
-U 1 1 62491CE2
-P 9150 1850
-F 0 "R?" V 8943 1850 50  0000 C CNN
-F 1 "R" V 9034 1850 50  0000 C CNN
-F 2 "" V 9080 1850 50  0001 C CNN
-F 3 "~" H 9150 1850 50  0001 C CNN
-	1    9150 1850
-	0    1    1    0
-$EndComp
 Text GLabel 9000 1850 0    50   Input ~ 0
 GND
 Text GLabel 9000 1750 0    50   Input ~ 0
-AT_D5
+AT_P12
 Wire Wire Line
 	9000 1750 9300 1750
@@
 	1    0    0    -1
 $EndComp
-$Comp
-L Device:R R?
-U 1 1 6249307C
-P 9150 2300
-F 0 "R?" V 8943 2300 50  0000 C CNN
-F 1 "R" V 9034 2300 50  0000 C CNN
-F 2 "" V 9080 2300 50  0001 C CNN
-F 3 "~" H 9150 2300 50  0001 C CNN
-	1    9150 2300
-	0    1    1    0
-$EndComp
 Text GLabel 9000 2300 0    50   Input ~ 0
 GND
 Text GLabel 9000 2200 0    50   Input ~ 0
-AT_D6
+AT_P4
 Wire Wire Line
 	9000 2200 9300 2200
@@
 	1    0    0    -1
 $EndComp
-$Comp
-L Device:R R?
-U 1 1 62494160
-P 9150 2700
-F 0 "R?" V 8943 2700 50  0000 C CNN
-F 1 "R" V 9034 2700 50  0000 C CNN
-F 2 "" V 9080 2700 50  0001 C CNN
-F 3 "~" H 9150 2700 50  0001 C CNN
-	1    9150 2700
-	0    1    1    0
-$EndComp
 Text GLabel 9000 2700 0    50   Input ~ 0
 GND
 Text GLabel 9000 2600 0    50   Input ~ 0
-PC?
+AT_P5
 Wire Wire Line
 	9000 2600 9300 2600
@@
 	1    0    0    -1
 $EndComp
-$Comp
-L Device:R R?
-U 1 1 624955FD
-P 9150 3100
-F 0 "R?" V 8943 3100 50  0000 C CNN
-F 1 "R" V 9034 3100 50  0000 C CNN
-F 2 "" V 9080 3100 50  0001 C CNN
-F 3 "~" H 9150 3100 50  0001 C CNN
-	1    9150 3100
-	0    1    1    0
-$EndComp
 Text GLabel 9000 3100 0    50   Input ~ 0
 GND
 Text GLabel 9000 3000 0    50   Input ~ 0
-PC?
+AT_P6
 Wire Wire Line
 	9000 3000 9300 3000
@@
 $EndComp
 Text GLabel 8400 4200 0    50   Input ~ 0
-AT_D11
+AT_P7
 $Comp
 L Connector:Screw_Terminal_01x02 SW_OP_SCREW
@@
 $EndComp
 Text GLabel 8400 5600 0    50   Input ~ 0
-AT_D12
+AT_P8
 $Comp
 L Connector:Screw_Terminal_01x02 SW_CL_SCREW
@@
 $EndComp
 Text GLabel 11400 800  0    50   Input ~ 0
-V5
+GND
 Wire Wire Line
 	11400 800  11850 800
@@
 	11850 900  11400 900
 Text GLabel 11400 900  0    50   Input ~ 0
-AT_D12
+AT_P9
 $Comp
 L Connector:Screw_Terminal_01x02 J?
@@
 	11850 1450 11400 1450
 Text GLabel 11400 1450 0    50   Input ~ 0
-AT_D13
+AT_P10
 $Comp
 L Own:RF_RX_433MHz U?
@@
 GND
 Text GLabel 11550 2150 0    50   Input ~ 0
-AT_D14
+AT_P11
 Text GLabel 12250 2050 2    50   Input ~ 0
 V5
@@
 $EndComp
 Text GLabel 6650 4050 2    50   Input ~ 0
-AT_D11
+AT_P5
 Text GLabel 6650 4150 2    50   Input ~ 0
-AT_D12
+AT_P6
 Wire Wire Line
 	6500 4050 6650 4050
@@
 	6500 4150 6650 4150
 Text GLabel 6650 4250 2    50   Input ~ 0
-AT_D13
+AT_P7
 Wire Wire Line
 	6500 4250 6650 4250
 Text GLabel 6650 1850 2    50   Input ~ 0
-AT_D14
+AT_P8
 Wire Wire Line
 	6650 1850 6500 1850
+Text GLabel 6650 1950 2    50   Input ~ 0
+AT_P9
+Text GLabel 6650 2050 2    50   Input ~ 0
+AT_P10
+Wire Wire Line
+	6500 1950 6650 1950
+Wire Wire Line
+	6500 2050 6650 2050
+Text GLabel 6650 2150 2    50   Input ~ 0
+AT_P11
+Wire Wire Line
+	6500 2150 6650 2150
+Wire Wire Line
+	6500 2350 7050 2350
+Wire Wire Line
+	7050 2350 7050 1500
+Wire Wire Line
+	7050 1500 7400 1500
+$Comp
+L Device:LED D?
+U 1 1 6246F5BE
+P 7550 1500
+F 0 "D?" H 7543 1245 50  0000 C CNN
+F 1 "LED" H 7543 1336 50  0000 C CNN
+F 2 "" H 7550 1500 50  0001 C CNN
+F 3 "~" H 7550 1500 50  0001 C CNN
+	1    7550 1500
+	-1   0    0    1
+$EndComp
+$Comp
+L Device:R R?
+U 1 1 62470486
+P 7950 1500
+F 0 "R?" V 7743 1500 50  0000 C CNN
+F 1 "1k" V 7834 1500 50  0000 C CNN
+F 2 "" V 7880 1500 50  0001 C CNN
+F 3 "~" H 7950 1500 50  0001 C CNN
+	1    7950 1500
+	0    1    1    0
+$EndComp
+Wire Wire Line
+	7700 1500 7800 1500
+Text GLabel 8200 1500 2    50   Input ~ 0
+GND
+Wire Wire Line
+	8100 1500 8200 1500
+Wire Wire Line
+	9000 1400 9300 1400
+Wire Wire Line
+	9000 1850 9300 1850
+Wire Wire Line
+	9000 2300 9300 2300
+Wire Wire Line
+	9000 2700 9300 2700
+Wire Wire Line
+	9000 3100 9300 3100
 $EndSCHEMATC

Commit message: Update
Parts:
- removed J?: Screw_Terminal_01x02, symbol Connector:Screw_Terminal_01x02
- added AT_OBST_SCREW1: Screw_Terminal_01x03, TerminalBlock:TerminalBlock_bornier-3_P5.08mm, symbol Connector:Screw_Terminal_01x03
- AT_328P1: renamed from U?; value ATmega328P-PU -> http://www.microchip.com/filehandler/redirect?http://ww1.microchip.com/downloads/en/DeviceDoc/ATmega328_P%20AVR%20MCU%2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
- AT_CLOSE1, AT_CLOSE_LIMIT1, AT_INDI_SCREW1, AT_OPEN1, AT_OPEN_LIMIT1, AT_STOP1, AT_UART_SCREW1: renamed from J?; footprint (none) -> TerminalBlock:TerminalBlock_bornier-2_P5.08mm
- AT_CLOSESW_Q1: renamed from SW_CL_Q; footprint (none) -> Package_TO_SOT_THT:TO-92; symbol Device:Q_NPN_BCE -> Transistor_BJT:BC337
- AT_CLOSESW_R1: renamed from SW_CL_Q; value R -> 16; footprint (none) -> Resistor_THT:R_Axial_DIN0204_L3.6mm_D1.6mm_P5.08mm_Horizontal
- AT_CLOSESW_SCREW1: renamed from SW_CL_SCREW; footprint (none) -> TerminalBlock:TerminalBlock_bornier-2_P5.08mm
- AT_LED1: renamed from D?; footprint (none) -> LED_THT:LED_D5.0mm
- AT_OPENSW_Q1: renamed from SW_OP_Q; footprint (none) -> Package_TO_SOT_THT:TO-92; symbol Device:Q_NPN_BCE -> Transistor_BJT:BC337
- AT_OPENSW_R1: renamed from SW_OP_R; value R -> 16; footprint (none) -> Resistor_THT:R_Axial_DIN0204_L3.6mm_D1.6mm_P5.08mm_Horizontal
- AT_OPENSW_SCREW1: renamed from SW_OP_SCREW; footprint (none) -> TerminalBlock:TerminalBlock_bornier-2_P5.08mm
- AT_R1: renamed from R?; footprint (none) -> Resistor_THT:R_Axial_DIN0204_L3.6mm_D1.6mm_P2.54mm_Vertical
- AT_RES_R1: renamed from AT_R1; footprint (none) -> Resistor_THT:R_Axial_DIN0204_L3.6mm_D1.6mm_P5.08mm_Horizontal
- AT_RES_SW1: renamed from AT_SW_R; footprint (none) -> Button_Switch_THT:SW_PUSH_6mm
- AT_RF1: renamed from U?; footprint (none) -> Own:RF_RX_433MHz
- AT_V_C1: renamed from AT_C100U; footprint (none) -> Capacitor_THT:CP_Radial_D8.0mm_P5.00mm
- AT_XTAL1: renamed from AT_XTAL; footprint (none) -> Crystal:Resonator-2Pin_W6.0mm_H3.0mm
- AT_XTAL_C1: renamed from AT_C20P1; footprint (none) -> Capacitor_THT:CP_Radial_D8.0mm_P3.80mm
- AT_XTAL_C2: renamed from AT_C20P2; footprint (none) -> Capacitor_THT:CP_Radial_D8.0mm_P3.80mm
- MV_12V_7812: renamed from MV_U2; footprint (none) -> Package_TO_SOT_THT:TO-220-3_Vertical
- MV_12V_D1: renamed from MV_D2; footprint (none) -> Diode_THT:D_T-1_P5.08mm_Horizontal
- MV_5V_7805: renamed from MV_U1; footprint (none) -> Package_TO_SOT_THT:TO-220-3_Vertical
- MV_5V_C1: renamed from MV_C1; footprint (none) -> Capacitor_THT:CP_Radial_D8.0mm_P5.00mm
- MV_5V_D1: renamed from MV_D1; footprint (none) -> Diode_THT:D_T-1_P5.08mm_Horizontal
- MV_SCREW1: renamed from MV_SCREW; footprint (none) -> TerminalBlock:TerminalBlock_bornier-2_P5.08mm
Connections:
- net AT_P10: no longer AT_INDI_SCREW1.2 (Pin_2)
- net AT_P12: now also AT_328P1.18 (PB4); no longer AT_328P1.5 (PD3)
- net AT_P9: now also AT_INDI_SCREW1.1 (Pin_1)
- net GND: now also AT_INDI_SCREW1.2 (Pin_2), AT_OBST_SCREW1.3 (Pin_3)
- net V5: now also AT_OBST_SCREW1.1 (Pin_1); no longer AT_INDI_SCREW1.1 (Pin_1)
- net AT_PA0: now reaches AT_328P1.23 (PC0)
- net AT_PA0: now also AT_OBST_SCREW1.2 (Pin_2)
- net at AT_OPENSW_Q1.1 (C): now also AT_OPENSW_SCREW1.2 (Pin_2); no longer AT_OPENSW_R1.1
- net at AT_OPENSW_Q1.2 (B): now also AT_OPENSW_R1.1; no longer AT_OPENSW_SCREW1.2 (Pin_2)
- net at AT_CLOSESW_Q1.1 (C): now also AT_CLOSESW_SCREW1.2 (Pin_2); no longer AT_CLOSESW_R1.1
- net at AT_CLOSESW_Q1.2 (B): now also AT_CLOSESW_R1.1; no longer AT_CLOSESW_SCREW1.2 (Pin_2)
Other:
- note added: "MV - Module Voltage"
- moved on the sheet: AT_INDI_SCREW1, AT_RF1
